File: robopoly_shield.brd (EAGLE design)
At the start: 50 x 50 mm, 39 parts, among them CON1 4UCON-19836, CON2 4UCON-10679, IC1 BLUETOOTH, IC2 DRV8833PWPR, X1 MICROMATCH-4

Commit message: Updated everything
Parts:
- removed POT1: 10K, karl_new:B25P
- removed SJ2, SJ4, SJ7: (no value), robopoly:SJ
- added JP3: JUMPER, robopoly:JUMPER
- added LED1: LED, led:CHIPLED_0805
- added POT: 10K, robopoly:B25P
- added R14, R15: 10K, rcl:R0805
- IC1: value BLUETOOTH -> DRV8833PWPR; device robopoly:BLUETOOTH -> robopoly:HTSSOP-16
- IC2: value DRV8833PWPR -> BLUETOOTH; device robopoly:HTSSOP-16 -> robopoly:BLUETOOTH
- LED2: device karl:CHIPLED_0805 -> led:CHIPLED_0805
- R5: value 330R -> 10K
- R7, R8: value 10K -> 1K
- X1: device karl_new:MICROMATCH-4 -> robopoly:MICROMATCH-4
- moved R8 38.6 mm to (2.00, 46.5), turned to 270 degrees
- moved R5 36.2 mm to (4.00, 8.50), flipped to the bottom, turned to 180 degrees
- moved R7 34.4 mm to (25.0, 34.5), flipped to the top
- moved IC1 22.0 mm to (12.0, 31.0), flipped to the top, turned to 270 degrees
- moved IC2 22.0 mm to (32.6, 38.7), flipped to the bottom, turned to 90 degrees
- moved R6 14.7 mm to (31.0, 12.0), turned to 0 degrees
- moved R1 8.31 mm to (36.4, 28.8), turned to 180 degrees
- moved R4 8.31 mm to (36.4, 21.2), turned to 180 degrees
- moved U$9 3.00 mm to (25.0, 37.5)
- moved R2 2.77 mm to (36.4, 26.3), turned to 180 degrees
- moved R3 2.77 mm to (36.4, 23.7), turned to 180 degrees
- renumbered BTN1 to BTN
Connections:
- removed net N$4: POT1.S, SJ7.1
- removed net N$9: R5.2, SJ4.2
- new net LED: PIN1.26, R8.2
- new net N$1: POT.S, R6.2
- new net N$12: JP3.A, R6.1
- new net N$13: LED1.A, R8.1
- net 3V3: now also IC2.12; no longer IC1.12
- net AIN1: now also IC1.15; no longer IC2.15
- net AIN2: now also IC1.16; no longer IC2.16
- net AOUT1: now also IC1.2; no longer IC2.2
- net AOUT2: now also IC1.4; no longer IC2.4
- net BIN1: now also IC1.9; no longer IC2.9
- net BIN2: now also IC1.10; no longer IC2.10
- net BOUT1: now also IC1.7; no longer IC2.7
- net BOUT2: now also IC1.5; no longer IC2.5
- net BUTTON: now also R5.2; no longer R8.2, SJ2.2
- net BUZZER: now also R7.2; no longer SJ4.1
- net GND: now also IC1.3, IC1.6, IC1.PAD@1, IC1.PAD@2, IC1.PAD@3, IC1.PAD@4, IC1.PAD@5, IC1.PAD@6, IC1.PAD@7, IC1.PAD@8, IC2.14, IC2.21, IC2.22, LED1.C, POT.A, R1.1, R2.1, R3.1, R4.1; no longer IC1.14, IC1.21, IC1.22, IC2.3, IC2.6, IC2.PAD@1, IC2.PAD@2, IC2.PAD@3, IC2.PAD@4, IC2.PAD@5, IC2.PAD@6, IC2.PAD@7, IC2.PAD@8, POT1.A, R1.2, R2.2, R3.2, R4.2
- net N$18: now also R5.1; no longer SJ2.1
- net N$2: now also IC2.31; no longer IC1.31
- net N$27: now also IC2.2; no longer IC1.2
- net N$5: now also IC1.14; no longer IC2.14
- net N$6: now also IC1.11; no longer IC2.11
- net N$7: now also R7.1; no longer R5.1
- net N$8: now also IC2.34; no longer IC1.34
- net POT: now also JP3.B; no longer SJ7.2
- net RX: now also R3.2; no longer R2.1
- net SCL: now also R1.2, R14.1; no longer R4.1, R6.1
- net SDA: now also R15.1, R2.2; no longer R3.1, R7.1
- net TX: now also IC2.1, R4.2; no longer IC1.1, R1.1
- net VCC: now also IC1.1, POT.E, R14.2, R15.2; no longer IC2.1, POT1.E, R6.2, R7.2, R8.1
- net VM: now also IC1.12; no longer IC2.12
Routing:
- net LED: track 0.00 -> 10.8 mm
- net N$4: track 8.70 -> 0.00 mm
- net N$12: track 0.00 -> 6.94 mm
- net N$9: track 5.69 -> 0.00 mm
- net VCC: track 129.2 -> 124.6 mm, vias 2 -> 1
- net BUZZER: track 13.9 -> 16.7 mm
- net N$1: track 0.00 -> 2.59 mm
- net SCL: track 48.1 -> 46.6 mm
- net SDA: track 55.7 -> 54.8 mm
- net BUTTON: track 59.8 -> 59.0 mm
- net N$13: track 0.00 -> 0.10 mm, vias 0 -> 1
Other:
- outline, holes or cut-outs redrawn
- board text added: "BTN/7"
- board text added: "BZR/8"
- board text added: "I C"
- board text added: "Kangur - 2014"
- board text added: "R14"
- board text added: "R15"
- board text added: "S1"
- board text added: "S1/6"
- board text added: "S2"
- board text added: "S2/5"
- board text added: "Ver. 2"
- board text removed: "5"
- board text removed: "6"
- board text removed: "7"
- board text removed: "8"
- board text removed: "I2C"
- board text removed: "Kangur - 2013"
- board text removed: "POT"
- board text removed: "Ver. 1"

Commit message: Replaced 4 channel DIP-switch with 2 and added stackable SPI header
Parts:
- removed R14, R15: 10K, rcl:R0805
- added ISP1: ISP-6PIN, robopoly:2X3-NOSILK-STACK
- PIN1: value ARDUINO-SMALL -> ARDUINOSTACK; device robopoly:ARDUINO-SMALL -> robopoly:ARDUINO-LONG
- R11: value 1K -> 2K
- R12: value 2K -> 10K
- R13: value 1K -> 10K
- R5, R6: value 10K -> 1K
- SW1: value (none) -> SW_DIP-2; device robopoly:EDG-04 -> robopoly:EDG-02
- moved R6 45.1 mm to (2.00, 46.5), turned to 270 degrees
- moved R8 40.9 mm to (42.5, 41.0), flipped to the top, turned to 90 degrees
- moved R3 35.8 mm to (4.00, 8.50)
- moved R13 35.3 mm to (45.0, 6.50), flipped to the bottom, turned to 180 degrees
- moved R5 33.4 mm to (25.0, 34.5), flipped to the top
- moved R7 23.4 mm to (47.5, 41.0), turned to 90 degrees
- moved R12 20.9 mm to (45.0, 16.5), flipped to the bottom, turned to 180 degrees
- moved R4 10.6 mm to (31.0, 12.0), turned to 0 degrees
- moved R9 10.0 mm to (37.5, 41.0)
- moved R11 7.07 mm to (37.5, 36.0)
- moved SW1 7.00 mm to (37.0, 25.0), turned to 0 degrees
- moved R1 4.25 mm to (38.3, 25.0), turned to 90 degrees
- moved R2 1.43 mm to (35.7, 25.0), turned to 90 degrees
Connections:
- net BTAT: now also R9.2; no longer R13.2
- net BUTTON: now also R3.2; no longer R5.2
- net BUZZER: now also R5.2; no longer R7.2
- net GND: now also ISP1.6, R1.2, R11.1, R2.2; no longer R1.1, R12.1, R2.1, R3.1, R4.1
- net LED: now also R6.2; no longer R8.2
- net N$1: now also R4.2; no longer R6.2
- net N$12: now also R4.1; no longer R6.1
- net N$13: now also R6.1; no longer R8.1
- net N$18: now also R3.1; no longer R5.1
- net N$2: now also R8.2; no longer R11.2
- net N$27: now also R7.1; no longer R9.1
- net N$3: now also R8.1; no longer R11.1
- net N$7: now also R5.1; no longer R7.1
- net N$8: now also R11.2, R9.1; no longer R12.2, R13.1
- net RX: now also R1.1, R7.2, SW1.2; no longer R3.2, R9.2, SW1.7
- net SCL: now also R12.1; no longer R1.2, R14.1, SW1.5
- net SDA: now also R13.1; no longer R15.1, R2.2, SW1.6
- net TX: now also R2.1, SW1.1; no longer R4.2, SW1.8
- net VCC: now also R12.2, R13.2; no longer R14.2, R15.2, SW1.1, SW1.2
Routing:
- net SDA: track 54.8 -> 48.4 mm
- net RX: track 34.3 -> 37.2 mm, vias 0 -> 1
- net SCL: track 46.6 -> 43.7 mm
- net VCC: track 124.6 -> 126.4 mm
- net N$27: track 14.4 -> 12.7 mm
- net TX: track 42.6 -> 43.2 mm, vias 1 -> 0
Other:
- board text added: "2014-02-10"
- board text added: "DIP"
- board text added: "H-BRIDGE"
- board text added: "Licence: CC-BY"
- board text added: "POT"
- board text added: "POWER"
- board text added: "Robopoly Shield"
- board text added: "SERVO"
- board text added: "SPI"
- board text added: "Version: 2"
- board text added: "http://robopoly.epfl.ch"
- board text removed: "DIP Switch"
- board text removed: "H-bridge"
- board text removed: "Pot"
- board text removed: "Power"
- board text removed: "R14"
- board text removed: "R15"
- board text removed: "Servo"

Commit message: Final update for this version... probably
Parts:
- added CON3: 4UCON-19963, robopoly:4UCON-19963
- added SJ2: (no value), robopoly:SJ
- CON2: value 4UCON-10679 -> 4UCON-19963; device robopoly:4UCON-10679 -> robopoly:4UCON-19963
- moved CON2 3.50 mm to (0.00, 29.5)
- moved R5 2.00 mm to (27.0, 34.5)
- moved LED2 1.00 mm to (42.5, 35.0)
- moved R10 1.00 mm to (47.5, 35.0)
- moved R11 1.00 mm to (37.5, 35.0)
- moved R7 1.00 mm to (47.5, 40.0)
- moved R8 1.00 mm to (42.5, 40.0)
- moved R9 1.00 mm to (37.5, 40.0)
Connections:
- new net N$9: R5.2, SJ2.1
- net AOUT1: now also CON3.1; no longer CON2.1
- net AOUT2: now also CON3.2; no longer CON2.2
- net BOUT1: now also CON2.2; no longer CON2.4
- net BOUT2: now also CON2.1; no longer CON2.3
- net BUZZER: now also SJ2.2; no longer R5.2
Routing:
- net AOUT2: track 6.85 -> 1.52 mm
- net BOUT1: track 6.00 -> 2.47 mm
- net AOUT1: track 8.40 -> 5.14 mm
- net N$9: track 0.00 -> 2.34 mm
- net N$8: track 12.3 -> 13.3 mm
- net N$4: track 0.00 -> 1.00 mm
- net N$2: track 7.05 -> 8.05 mm
- net BTAT: track 8.36 -> 9.36 mm
- net N$7: track 12.0 -> 11.2 mm
- net BOUT2: track 5.84 -> 5.02 mm
- net BUZZER: track 16.7 -> 16.0 mm
- net RX: track 37.2 -> 37.8 mm
- net TX: track 43.2 -> 43.8 mm
Other:
- board text added: "2014-07-25"
- board text removed: "2014-02-10"
